Commit message: add pinocchio code Cmakelist templete

File: C++/RBDL_Eigen_Example/example/URDF/simple_manipulator.urdf (robot description, URDF)
Before this commit: robot simple_manipulator, 4 links, 3 joints
Links:
- link base_link: mass 0.1 -> 0.0; geometry collision box size=0.05 0.05 0.2; visual box size=0.0 0.0 0.0
Joints:
- joint Joint1: origin xyz=0.0 0.0 0.225 rpy=0.0 0.0 0.0 -> xyz=0.0 0.0 0.0 rpy=0.0 0.0 0.0
